File: 01.brd (EAGLE design)
At the start: 48 x 72 mm, 10 parts, among them U1 I-06220_ATP3011F1-PU, U2 KONASHI

Commit message: add .gitignore
Parts:
- removed C2: (no value), MyPacklbr:C0603
- added C4: (no value), MyPacklbr:C0603
- moved R2 9.01 mm to (3.84, 28.0)
- moved C3 6.00 mm to (19.0, 43.9)
- moved R1 2.92 mm to (3.89, 24.4)
- moved U1 1.12 mm to (11.1, 43.4)
Connections:
- removed net N$1: C1.2, C1.3, C1.4, C1.5, C2.2
- net GND: now also C4.2, U2.20
- net N$2: now also C1.2, C1.3, C1.4, C1.5, C4.1; no longer C2.1
Routing:
- net GND: track 114.2 -> 0.00 mm
- net +3V3: track 229.1 -> 129.3 mm
- net N$5: track 65.1 -> 38.5 mm
- net N$1: track 21.7 -> 0.00 mm
- net N$8: track 48.9 -> 33.6 mm
- net N$2: track 29.4 -> 42.0 mm
- added copper zone on layer 1, net GND
- removed copper zone on layer 1, net N$3
